Commit message: Added a robotic arm to be added on top of mobile robot

File: src/my_robot_description/urdf/common_properties.xacro (robot description, xacro)
@@ -6,4 +6,10 @@
     <material name="grey">
         <color rgba="0.5 0.5 0.5 1" />
+    </material>
+    <material name="orange">
+        <color rgba="0.96 0.58 0.15 1" />
+    </material>
+    <material name="yellow">
+        <color rgba="0.96 0.99 0.08 1" />
     </material>
     <xacro:macro name="box_inertia" params="m l w h xyz rpy">
