Commit message: Added collision adn inertia tags to be able to run on gazebo

File: src/my_robot_description/urdf/arm.xacro (robot description, xacro)
@@ -1,28 +1,79 @@
 <?xml version="1.0"?>
-<robot name="my_robot" xmlns:xacro="http:s//www.ros.org/wiki/xacro">
+<robot xmlns:xacro="http:s//www.ros.org/wiki/xacro">
+    <xacro:property name="arm_base_length" value="0.1" />
     <xacro:property name="arm_base_width" value="0.1" />
     <xacro:property name="arm_base_height" value="0.02" />
+    <xacro:property name="forearm_length" value="0.3" />
+    <xacro:property name="forearm_radius" value="0.02" />
+    <xacro:property name="hand_length" value="0.3" />
+    <xacro:property name="hand_radius" value="0.02" />
     <link name="arm_base_link">
         <visual>
             <geometry>
-                <box size="0.1 ${arm_base_width} 0.02" />
+                <box size="${arm_base_length} ${arm_base_width} ${arm_base_height}" />
             </geometry>
-            <origin xyz="0 0 0" rpy="0 0 0" />
+            <origin xyz="0 0 ${arm_base_height / 2.0}" rpy="0 0 0" />
             <material name="orange" />
         </visual>
         <collision>
-            <origin xyz="0 0 0" rpy="0 0 0" />
+            <origin xyz="0 0 ${arm_base_height / 2.0}" rpy="0 0 0" />
             <geometry>
-                <box size="0.1 0.1 0.02" />
+                <box size="${arm_base_length} ${arm_base_width} ${arm_base_height}" />
             </geometry>
         </collision>
-        <xacro:box_inertia m="0.5" l="0.1" w="0.1" h="0.02" xyz="0 0 0" rpy="0 0 0" />
+        <xacro:box_inertia m="0.5" l="${2*arm_base_length}" w="${2*arm_base_width}"
+            h="${2*arm_base_height}" xyz="0 0 ${arm_base_height / 2.0}" rpy="0 0 0" />
     </link>
-    <link name="base_footprint">
+    <link name="forearm_link">
+        <visual>
+            <geometry>
+                <cylinder radius="${forearm_radius}" length="${forearm_length}" />
+            </geometry>
+            <origin xyz="0 0 ${forearm_length / 2}" rpy="0 0 0" />
+            <material name="yellow" />
+        </visual>
+        <collision>
+            <origin xyz="0 0 ${forearm_length / 2}" rpy="0 0 0" />
+            <geometry>
+                <cylinder radius="${forearm_radius}" length="${forearm_length}" />
+            </geometry>
+        </collision>
+        <xacro:cylinder_inertia m="0.3" r="${2*forearm_radius}" h="${2*forearm_length}"
+            xyz="0 0 ${forearm_length / 2}"
+            rpy="0 0 0" />
     </link>
-    <joint name="base_arm_joint" type="fixed">
-        <parent link="base_footprint" />
-        <child link="arm_base_link" />
-        <origin xyz="0 0 ${arm_base_height / 2}" rpy="0 0 0" />
+    <link name="hand_link">
+        <visual>
+            <geometry>
+                <cylinder radius="${hand_radius}" length="${hand_length}" />
+            </geometry>
+            <origin xyz="0 0 ${hand_length / 2.0}" rpy="0 0 0" />
+            <material name="orange" />
+        </visual>
+        <collision>
+            <origin xyz="0 0 ${hand_length / 2.0}" rpy="0 0 0" />
+            <geometry>
+                <cylinder radius="${hand_radius}" length="${hand_length}" />
+            </geometry>
+        </collision>
+        <xacro:cylinder_inertia m="0.3" r="${2*hand_radius}" h="${2*hand_length}"
+            xyz="0 0 ${hand_length / 2.0}"
+            rpy="0 0 0" />
+    </link>
+    <joint name="arm_base_forearm_joint" type="revolute">
+        <parent link="arm_base_link" />
+        <child link="forearm_link" />
+        <origin xyz="0 0 ${arm_base_height}" rpy="0 0 0" />
+        <limit lower="0" upper="${pi / 2}" effort="100" velocity="100" />
+        <dynamics friction="0.05" damping="0.1" />
+        <axis xyz="0 1 0" />
+    </joint>
+    <joint name="forearm_hand_joint" type="revolute">
+        <parent link="forearm_link" />
+        <child link="hand_link" />
+        <origin xyz="0 0 ${forearm_length}" rpy="0 0 0" />
+        <limit lower="0" upper="${pi / 2}" effort="100" velocity="100" />
+        <dynamics friction="0.05" damping="0.1" />
+        <axis xyz="0 1 0" />
     </joint>
 </robot>

File: src/my_robot_description/urdf/common_properties.xacro (robot description, xacro)
@@ -8,8 +8,8 @@
     </material>
     <material name="orange">
-        <color rgba="0.96 0.58 0.15 1" />
+        <color rgba="1.0 0.5 0 1" />
     </material>
     <material name="yellow">
-        <color rgba="0.96 0.99 0.08 1" />
+        <color rgba="1.0 1.0 0 1" />
     </material>
     <xacro:macro name="box_inertia" params="m l w h xyz rpy">

File: src/my_robot_description/urdf/mobile_base_gazebo.xacro (robot description, xacro)
@@ -36,3 +36,20 @@
         </plugin>
     </gazebo>
+    <gazebo>
+        <plugin name="joint_state_publisher"
+            filename="libgazebo_ros_joint_state_publisher.so">
+            <!-- Update rate in Hertz -->
+            <update_rate>10</update_rate>
+            <!-- Name of joints in the model whose states will be published. -->
+            <joint_name>arm_base_forearm_joint</joint_name>
+            <joint_name>forearm_hand_joint</joint_name>
+        </plugin>
+    </gazebo>
+    <gazebo>
+        <plugin name="joint_pose_trajectory"
+            filename="libgazebo_ros_joint_pose_trajectory.so">
+            <!-- Update rate in Hz -->
+            <update_rate>2</update_rate>
+        </plugin>
+    </gazebo>
 </robot>

File: src/my_robot_description/urdf/standalone_arm.urdf.xacro (robot description, xacro)
@@ -3,36 +3,4 @@
     <xacro:include filename="common_properties.xacro" />
     <xacro:include filename="arm.xacro" />
-    <xacro:property name="length_of_arm" value="0.3" />
-    <link name="forearm_link">
-        <visual>
-            <geometry>
-                <cylinder radius="0.02" length="${length_of_arm}" />
-            </geometry>
-            <origin xyz="0 0 ${arm_base_height / 2}" rpy="0 0 0" />
-            <material name="yellow" />
-        </visual>
-    </link>
-    <link name="hand_link">
-        <visual>
-            <geometry>
-                <cylinder radius="0.02" length="${length_of_arm}" />
-            </geometry>
-            <origin xyz="0 0 ${(length_of_arm + arm_base_height) / 2}" rpy="0 0 0" />
-            <material name="orange" />
-        </visual>
-    </link>
-    <joint name="arm_base_forearm_joint" type="revolute">
-        <parent link="arm_base_link" />
-        <child link="forearm_link" />
-        <origin xyz="0 0 ${length_of_arm / 2}" rpy="0 0 0" />
-        <limit lower="0" upper="${pi / 2}" effort="100" velocity="100" />
-        <dynamics friction="0.05" damping="0.1" />
-    </joint>
-    <joint name="forearm_hand_joint" type="revolute" >
-        <parent link="forearm_link" />
-        <child link="hand_link" />
-        <origin xyz="0 0 ${length_of_arm / 2}" rpy="0 0 0" />
-        <limit lower="0" upper="${pi / 2}" effort="100" velocity="100" />
-        <dynamics friction="0.05" damping="0.1" />
-    </joint>
+    <xacro:include filename="arm_gazebo.xacro" />
 </robot>
